File: NokiaLCD_shield/_autosave-Arduino_UNO_Shield_Template.kicad_pcb (KiCad board)
At the start: 2 copper layers, 72.7 x 53.4 mm, 13 parts, among them CON1 Nokia1616_LCD, P1 CONN_01X02, Q1 BC547_BEC_123, U1 ArduinoUnoR3

Commit message: Changed Nokia1616 LCD backlight Added a low switch NPN transistor for PWM switching of backlight to ground Added a capacitor to ground on the 3v3 line Cleaned up the traces a bit
Changed lines of the file:
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@@
     (links 41)
     (no_connects 2)
-    (area 44.589699 72.440799 117.690901 126.174501)
+    (area 44.270239 72.440799 117.690901 126.174501)
     (thickness 1.6002)
     (drawings 6)
@@
     (visible_elements 7FFFEFFF)
     (pcbplotparams
-      (layerselection 0x00000_00000001)
+      (layerselection 0x00000_80000000)
       (usegerberextensions false)
       (excludeedgelayer false)
@@
       (subtractmaskfromsilk false)
       (outputformat 5)
-      (mirror true)
+      (mirror false)
       (drillshape 2)
       (scaleselection 1)
@@
   )
   (gr_line (start 117.5004 72.6313) (end 117.49024 125.95098) (angle 90) (layer Edge.Cuts) (width 0.381))
-  (gr_text DIGITAL (at 89.916 77.724 180) (layer F.SilkS)
+  (gr_text DIGITAL (at 89.916 77.724 -180) (layer F.SilkS)
     (effects (font (size 0.9144 1.016) (thickness 0.1016)))
   )
-  (gr_text DIGITAL (at 65.786 77.724 180) (layer F.SilkS)
+  (gr_text DIGITAL (at 65.786 77.724 -180) (layer F.SilkS)
     (effects (font (size 0.9144 1.016) (thickness 0.1016)))
   )
