File: voltage_divider/voltage_divider.sch (KiCad schematic (older format))
At the start: 3 parts

Commit message: Clean up the simulation folders
Remove a duplicate amplifier simulation project amplifier in favor of the opamp of the project
Remove uneccesary files in the opamp
Add a README.md to explain how to use the RC circuit simulation netlist file for the filter's characteristics and sample signal input and output
Parts:
- R1, R2: symbol R -> device:R
- v1: symbol CONN_01X02 -> voltage_divider-rescue:CONN_01X02-RESCUE-voltage_divider
Changed lines of the file:
@@
-EESchema Schematic File Version 2
-LIBS:power
-LIBS:device
-LIBS:transistors
-LIBS:conn
-LIBS:linear
-LIBS:regul
-LIBS:74xx
-LIBS:cmos4000
-LIBS:adc-dac
-LIBS:memory
-LIBS:xilinx
-LIBS:microcontrollers
-LIBS:dsp
-LIBS:microchip
-LIBS:analog_switches
-LIBS:motorola
-LIBS:texas
-LIBS:intel
-LIBS:audio
-LIBS:interface
-LIBS:digital-audio
-LIBS:philips
-LIBS:display
-LIBS:cypress
-LIBS:siliconi
-LIBS:opto
-LIBS:atmel
-LIBS:contrib
-LIBS:valves
+EESchema Schematic File Version 4
 LIBS:voltage_divider-cache
-EELAYER 25 0
+EELAYER 26 0
 EELAYER END
 $Descr A4 11693 8268
@@
 $EndDescr
 $Comp
-L R R2
+L device:R R2
 U 1 1 58D5003A
 P 5500 3900
@@
 $EndComp
 $Comp
-L R R1
+L device:R R1
 U 1 1 58D500BD
 P 5050 3600
@@
 $EndComp
 $Comp
-L CONN_01X02 v1
+L voltage_divider-rescue:CONN_01X02-RESCUE-voltage_divider v1
 U 1 1 58D50985
 P 4500 3800
