File: Arduino test/test.sch (KiCad schematic (older format))
At the start: 1 part, among them U1 ArduinoUnoR3

Commit message: Too many untracked changes: LCD boards update and switch to KiCAD version 5
Update the Nokia LCD breakout boards
Add more KiCAD simulation projects
Update most projects to KiCAD version 5
Parts:
- U1: symbol ArduinoUnoR3 -> test-rescue:ArduinoUnoR3
Changed lines of the file:
@@
-EESchema Schematic File Version 2
-LIBS:power
-LIBS:device
-LIBS:transistors
-LIBS:conn
-LIBS:linear
-LIBS:regul
-LIBS:74xx
-LIBS:cmos4000
-LIBS:adc-dac
-LIBS:memory
-LIBS:xilinx
-LIBS:microcontrollers
-LIBS:dsp
-LIBS:microchip
-LIBS:analog_switches
-LIBS:motorola
-LIBS:texas
-LIBS:intel
-LIBS:audio
-LIBS:interface
-LIBS:digital-audio
-LIBS:philips
-LIBS:display
-LIBS:cypress
-LIBS:siliconi
-LIBS:opto
-LIBS:atmel
-LIBS:contrib
-LIBS:valves
-EELAYER 25 0
+EESchema Schematic File Version 4
+EELAYER 30 0
 EELAYER END
 $Descr A4 11693 8268
@@
 $EndDescr
 $Comp
-L ArduinoUnoR3 U1
+L test-rescue:ArduinoUnoR3 U1
 U 1 1 5897B6F2
 P 5105 2615
