File: BJT_amplifier/BJT_amplifier.sch (KiCad schematic (older format))
At the start: 5 parts, among them Q1 BC107B

Commit message: Clean up the simulation folders
Remove a duplicate amplifier simulation project amplifier in favor of the opamp of the project
Remove uneccesary files in the opamp
Add a README.md to explain how to use the RC circuit simulation netlist file for the filter's characteristics and sample signal input and output
Parts:
- Q1: symbol Q_NPN_EBC -> device:Q_NPN_EBC
- R1, R2: symbol R -> device:R
- v1, v2: symbol CONN_01X02 -> BJT_amplifier-rescue:CONN_01X02-RESCUE-BJT_amplifier
Connections:
- net 1 renamed vin
- net 2 renamed base
- net 3 renamed vcollector
- net 4 renamed vout
Other:
- note added: "+PSPICE\n.model BC107B NPN(Is=7.049f Xti=3 Eg=1.11 Vaf=59.59 Bf=381.7 Ise=59.74f\n+ Ne=1.522 Ikf=3.289 Nk=.5 Xtb=1.5 Br=2.359 Isc=192.9p Nc=1.954\n+ Ikr=7.807 Rc=1.427 Cjc=5.38p Mjc=.329 Vjc=.6218 Fc=.5 Cje=11.5p\n+ Mje=.2718 Vje=.5 Tr=10n Tf=438p Itf=5.716 Xtf=14.51 Vtf=10)\n* PHILIPS pid=bc107b case=TO18\n* 91-08-02 dsq\n\n.dc V2 0 10 0.1 V1 1.5 3.5 0.5 \n\n************\n.control\nrun\nplot v(v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"
- note removed: "+PSPICE\n.model BC107B NPN(Is=7.049f Xti=3 Eg=1.11 Vaf=59.59 Bf=381.7 Ise=59.74f\n+ Ne=1.522 Ikf=3.289 Nk=.5 Xtb=1.5 Br=2.359 Isc=192.9p Nc=1.954\n+ Ikr=7.807 Rc=1.427 Cjc=5.38p Mjc=.329 Vjc=.6218 Fc=.5 Cje=11.5p\n+ Mje=.2718 Vje=.5 Tr=10n Tf=438p Itf=5.716 Xtf=14.51 Vtf=10)\n\n.dc V2 0 10 0.1 V1 1.5 3.5 0.5 \n\n************\n.control\nrun\nplot v(4,3)/1k vs v(3) \n.endc\n************\n\n.end"
- moved on the sheet: Q1, R1, R2, v1, v2
Changed lines of the file:
@@
 EESchema Schematic File Version 2
 LIBS:power
-LIBS:device
-LIBS:transistors
-LIBS:conn
-LIBS:linear
-LIBS:regul
-LIBS:74xx
-LIBS:cmos4000
-LIBS:adc-dac
-LIBS:memory
-LIBS:xilinx
-LIBS:microcontrollers
-LIBS:dsp
-LIBS:microchip
-LIBS:analog_switches
-LIBS:motorola
-LIBS:texas
-LIBS:intel
-LIBS:audio
-LIBS:interface
-LIBS:digital-audio
-LIBS:philips
-LIBS:display
-LIBS:cypress
-LIBS:siliconi
-LIBS:opto
-LIBS:atmel
-LIBS:contrib
-LIBS:valves
 LIBS:BJT_amplifier-cache
 EELAYER 25 0
 EELAYER END
-$Descr A4 11693 8268
+$Descr User 6299 7874
 encoding utf-8
 Sheet 1 1
-Title ""
-Date ""
-Rev ""
-Comp ""
+Title "BJT Transistor Characteristics"
+Date "2018-04-24"
+Rev "0.1.2"
+Comp "KARIBE ELECTRONICS"
 Comment1 ""
-Comment2 ""
-Comment3 ""
-Comment4 ""
+Comment2 "karibe.co.ke"
+Comment3 "@muriukidavid"
+Comment4 "Drawn by: David Muriuki Karibe"
 $EndDescr
 $Comp
-L CONN_01X02 v1
+L BJT_amplifier-rescue:CONN_01X02-RESCUE-BJT_amplifier v1
 U 1 1 59366B5C
-P 4300 4150
-F 0 "v1" H 4300 4300 50  0000 C CNN
-F 1 "DC 12" V 4400 4150 50  0000 C CNN
-F 2 "" H 4300 4150 50  0001 C CNN
-F 3 "" H 4300 4150 50  0001 C CNN
-	1    4300 4150
+P 1450 5300
+F 0 "v1" H 1450 5450 50  0000 C CNN
+F 1 "DC 12" V 1550 5300 50  0000 C CNN
+F 2 "" H 1450 5300 50  0001 C CNN
+F 3 "" H 1450 5300 50  0001 C CNN
+	1    1450 5300
 	-1   0    0    -1
 $EndComp
-Text GLabel 5050 4200 3    60   Input ~ 0
+Text GLabel 2200 5350 3    60   Input ~ 0
 0
-Text GLabel 4500 4050 2    60   Input ~ 0
-1
-Text Notes 3950 3050 0    60   ~ 0
-+PSPICE\n.model BC107B   NPN(Is=7.049f Xti=3 Eg=1.11 Vaf=59.59 Bf=381.7 Ise=59.74f\n+               Ne=1.522 Ikf=3.289 Nk=.5 Xtb=1.5 Br=2.359 Isc=192.9p Nc=1.954\n+               Ikr=7.807 Rc=1.427 Cjc=5.38p Mjc=.329 Vjc=.6218 Fc=.5 Cje=11.5p\n+               Mje=.2718 Vje=.5 Tr=10n Tf=438p Itf=5.716 Xtf=14.51 Vtf=10)\n\n.dc V2 0 10 0.1 V1 1.5 3.5 0.5 \n\n************\n.control\nrun\nplot v(4,3)/1k vs v(3) \n.endc\n************\n\n.end
-Text GLabel 5100 3500 1    60   Input ~ 0
-3
+Text GLabel 1650 5200 2    60   Input ~ 0
+vin
+Text Notes 1100 4200 0    60   ~ 0
++PSPICE\n.model BC107B   NPN(Is=7.049f Xti=3 Eg=1.11 Vaf=59.59 Bf=381.7 Ise=59.74f\n+               Ne=1.522 Ikf=3.289 Nk=.5 Xtb=1.5 Br=2.359 Isc=192.9p Nc=1.954\n+               Ikr=7.807 Rc=1.427 Cjc=5.38p Mjc=.329 Vjc=.6218 Fc=.5 Cje=11.5p\n+               Mje=.2718 Vje=.5 Tr=10n Tf=438p Itf=5.716 Xtf=14.51 Vtf=10)\n*       PHILIPS     pid=bc107b  case=TO18\n*       91-08-02 dsq\n\n.dc V2 0 10 0.1 V1 1.5 3.5 0.5 \n\n************\n.control\nrun\nplot v(vout,vcollector)/1k vs v(vcollector) \n.endc\n************\n\n.end
+Text GLabel 2250 4650 1    60   Input ~ 0
+vcollector
 $Comp
-L R R1
+L device:R R1
 U 1 1 5936898A
-P 4500 3850
-F 0 "R1" V 4580 3850 50  0000 C CNN
-F 1 "1Meg" V 4500 3850 50  0000 C CNN
-F 2 "" V 4430 3850 50  0001 C CNN
-F 3 "" H 4500 3850 50  0001 C CNN
-	1    4500 3850
+P 1650 5000
+F 0 "R1" V 1730 5000 50  0000 C CNN
+F 1 "1Meg" V 1650 5000 50  0000 C CNN
+F 2 "" V 1580 5000 50  0001 C CNN
+F 3 "" H 1650 5000 50  0001 C CNN
+	1    1650 5000
 	-1   0    0    1
 $EndComp
-Text GLabel 4600 3700 1    60   Input ~ 0
-2
+Text GLabel 1750 4850 1    60   Input ~ 0
+base
 $Comp
-L R R2
+L device:R R2
 U 1 1 59368BD6
-P 5400 3500
-F 0 "R2" V 5480 3500 50  0000 C CNN
-F 1 "1k" V 5400 3500 50  0000 C CNN
-F 2 "" V 5330 3500 50  0001 C CNN
-F 3 "" H 5400 3500 50  0001 C CNN
-	1    5400 3500
+P 2550 4650
+F 0 "R2" V 2630 4650 50  0000 C CNN
+F 1 "1k" V 2550 4650 50  0000 C CNN
+F 2 "" V 2480 4650 50  0001 C CNN
+F 3 "" H 2550 4650 50  0001 C CNN
+	1    2550 4650
 	0    1    1    0
 $EndComp
 $Comp
-L CONN_01X02 v2
+L BJT_amplifier-rescue:CONN_01X02-RESCUE-BJT_amplifier v2
 U 1 1 59368BFF
-P 5750 4000
-F 0 "v2" H 5750 4150 50  0000 C CNN
-F 1 "DC 10" V 5850 4000 50  0000 C CNN
-F 2 "" H 5750 4000 50  0001 C CNN
-F 3 "" H 5750 4000 50  0001 C CNN
-	1    5750 4000
+P 2900 5150
+F 0 "v2" H 2900 5300 50  0000 C CNN
+F 1 "DC 10" V 3000 5150 50  0000 C CNN
+F 2 "" H 2900 5150 50  0001 C CNN
+F 3 "" H 2900 5150 50  0001 C CNN
+	1    2900 5150
 	1    0    0    -1
 $EndComp
-Text GLabel 5550 3750 2    60   Input ~ 0
-4
+Text GLabel 2700 4900 2    60   Input ~ 0
+vout
 $Comp
-L Q_NPN_EBC Q1
+L device:Q_NPN_EBC Q1
 U 1 1 5936CAC5
-P 4850 3700
-F 0 "Q1" H 5050 3750 50  0000 L CNN
-F 1 "BC107B" H 5050 3650 50  0000 L CNN
-F 2 "" H 5050 3800 50  0001 C CNN
-F 3 "" H 4850 3700 50  0001 C CNN
-	1    4850 3700
+P 2000 4850
+F 0 "Q1" H 2200 4900 50  0000 L CNN
+F 1 "BC107B" H 2200 4800 50  0000 L CNN
+F 2 "" H 2200 4950 50  0001 C CNN
+F 3 "" H 2000 4850 50  0001 C CNN
+	1    2000 4850
 	1    0    0    1
 $EndComp
 Wire Wire Line
-	4500 4200 5550 4200
+	1650 5350 2700 5350
 Wire Wire Line
-	5550 4200 5550 4050
+	2700 5350 2700 5200
 Wire Wire Line
-	5550 3500 5550 3950
+	2700 4650 2700 5100
 Wire Wire Line
-	4950 3500 5250 3500
+	2100 4650 2400 4650
 Wire Wire Line
-	4500 3700 4650 3700
+	1650 4850 1800 4850
 Wire Wire Line
-	4500 4000 4500 4100
+	1650 5150 1650 5250
 Wire Wire Line
-	4950 3900 4950 4200
-Connection ~ 4950 4200
+	2100 5350 2100 5050
+Connection ~ 2100 5350
 $EndSCHEMATC

Commit message: Too many untracked changes: LCD boards update and switch to KiCAD version 5
Update the Nokia LCD breakout boards
Add more KiCAD simulation projects
Update most projects to KiCAD version 5
Parts:
- Q1: symbol device:Q_NPN_EBC -> BJT_amplifier-rescue:device_Q_NPN_EBC
- R1, R2: symbol device:R -> BJT_amplifier-rescue:device_R
- v1, v2: symbol BJT_amplifier-rescue:CONN_01X02-RESCUE-BJT_amplifier -> BJT_amplifier-rescue:BJT_amplifier-rescue_CONN_01X02-RESCUE-BJT_amplifier
Changed lines of the file:
@@
-EESchema Schematic File Version 2
-LIBS:power
+EESchema Schematic File Version 4
 LIBS:BJT_amplifier-cache
-EELAYER 25 0
+EELAYER 30 0
 EELAYER END
 $Descr User 6299 7874
@@
 Date "2018-04-24"
 Rev "0.1.2"
-Comp "KARIBE ELECTRONICS"
+Comp "KARIBE (K) LTD"
 Comment1 ""
 Comment2 "karibe.co.ke"
 Comment3 "@muriukidavid"
-Comment4 "Drawn by: David Muriuki Karibe"
+Comment4 "Drawn by: Karibe David"
 $EndDescr
 $Comp
-L BJT_amplifier-rescue:CONN_01X02-RESCUE-BJT_amplifier v1
+L BJT_amplifier-rescue:BJT_amplifier-rescue_CONN_01X02-RESCUE-BJT_amplifier v1
 U 1 1 59366B5C
 P 1450 5300
@@
 vcollector
 $Comp
-L device:R R1
+L BJT_amplifier-rescue:device_R R1
 U 1 1 5936898A
 P 1650 5000
@@
 base
 $Comp
-L device:R R2
+L BJT_amplifier-rescue:device_R R2
 U 1 1 59368BD6
 P 2550 4650
@@
 $EndComp
 $Comp
-L BJT_amplifier-rescue:CONN_01X02-RESCUE-BJT_amplifier v2
+L BJT_amplifier-rescue:BJT_amplifier-rescue_CONN_01X02-RESCUE-BJT_amplifier v2
 U 1 1 59368BFF
 P 2900 5150
@@
 vout
 $Comp
-L device:Q_NPN_EBC Q1
+L BJT_amplifier-rescue:device_Q_NPN_EBC Q1
 U 1 1 5936CAC5
 P 2000 4850
@@
 $EndComp
 Wire Wire Line
-	1650 5350 2700 5350
+	1650 5350 2100 5350
 Wire Wire Line
 	2700 5350 2700 5200
@@
 	2100 5350 2100 5050
 Connection ~ 2100 5350
+Wire Wire Line
+	2100 5350 2700 5350
 $EndSCHEMATC
