File: Nokia1616_LCD/Nokia1616_LCD.sch (KiCad schematic (older format))
At the start: 3 parts, among them P1 CONN_01X08

Commit message: Changed Nokia1616 LCD backlight Added a low switch NPN transistor for PWM switching of backlight to ground Added a capacitor to ground on the 3v3 line Cleaned up the traces a bit
Parts:
- added Q1: BC547_BEC_123, TO_SOT_Packages_SMD:SOT-23, symbol BC547_BEC_123
- added R1: 1K, Resistors_SMD:R_1206, symbol R
Connections:
- net GND: now also Q1.2 (E)
- net LED: now also R1.2; no longer CONN1.10 (LED-)
- net VCC: no longer CONN1.11 (LED+), P1.8 (P8)
- new net: Q1.1 (B), R1.1
- new net 5V: CONN1.11 (LED+), P1.8 (P8)
- new net LED-: CONN1.10 (LED-), Q1.3 (C)
Changed lines of the file:
@@
 P 3080 1640
 F 0 "CONN1" H 3080 890 60  0000 C CNN
-F 1 "Nokia1616_LCD" H 3080 2090 60  0000 C CNN
+F 1 "Nokia1616_LCD" H 3090 2225 60  0000 C CNN
 F 2 "Connect:Nokia1616_LCD" H 3180 1640 60  0001 C CNN
 F 3 "" H 3180 1640 60  0001 C CNN
@@
 Connection ~ 2440 1750
 Text GLabel 3590 1300 2    47   Input ~ 0
-LED
+LED-
 Text GLabel 3590 1560 2    47   Input ~ 0
-VCC
+5V
 Text GLabel 1610 2010 2    47   Input ~ 0
 VCC
@@
 CLK
 Text GLabel 1610 1310 2    47   Input ~ 0
-VCC
+5V
 Text GLabel 1610 1710 2    47   Input ~ 0
 RESET
 Text GLabel 1610 1610 2    47   Input ~ 0
 LED
+$Comp
+L BC547_BEC_123 Q1
+U 1 1 58C99E38
+P 4515 1925
+F 0 "Q1" H 4715 2000 50  0000 L CNN
+F 1 "BC547_BEC_123" H 3870 2060 50  0000 L CNN
+F 2 "TO_SOT_Packages_SMD:SOT-23" H 4715 1850 50  0001 L CIN
+F 3 "" H 4515 1925 50  0000 L CNN
+	1    4515 1925
+	1    0    0    -1
+$EndComp
+Text GLabel 4615 1725 1    47   Input ~ 0
+LED-
+Text GLabel 4615 2125 3    47   Input ~ 0
+GND
+Text GLabel 4015 1925 0    47   Input ~ 0
+LED
+$Comp
+L R R1
+U 1 1 58C9A3B8
+P 4165 1925
+F 0 "R1" V 4245 1925 50  0000 C CNN
+F 1 "1K" V 4165 1925 50  0000 C CNN
+F 2 "Resistors_SMD:R_1206" V 4095 1925 50  0001 C CNN
+F 3 "" H 4165 1925 50  0000 C CNN
+	1    4165 1925
+	0    1    1    0
+$EndComp
 $EndSCHEMATC

Commit message: Added Simulation Circuits and POV board
Added a BJT characteristics simulation circuit
Add a Voltage Divider simulation circuit
Add an amplifier simulation circuit
Add a Nokia LCD breakout board
Add a POV LED MKL05Z board
Parts:
- added P2: CONN_01X08, Pin_Headers:Pin_Header_Straight_1x08, symbol CONN_01X08
Connections:
- net 5V: now also P2.1 (P1)
- net CE: now also P2.6 (P6)
- net CLK: now also P2.2 (P2)
- net GND: now also P2.7 (P7)
- net LED: now also P2.4 (P4)
- net MOSI: now also P2.3 (P3)
- net RESET: now also P2.5 (P5)
- net VCC: now also P2.8 (P8)
Changed lines of the file:
@@
 	0    1    1    0
 $EndComp
+$Comp
+L CONN_01X08 P2
+U 1 1 58D4DEA8
+P 760 1660
+F 0 "P2" H 760 2110 50  0000 C CNN
+F 1 "CONN_01X08" V 860 1660 50  0000 C CNN
+F 2 "Pin_Headers:Pin_Header_Straight_1x08" H 760 1660 50  0001 C CNN
+F 3 "" H 760 1660 50  0000 C CNN
+	1    760  1660
+	-1   0    0    1
+$EndComp
+Text GLabel 960  1310 2    47   Input ~ 0
+VCC
+Text GLabel 960  1410 2    47   Input ~ 0
+GND
+Text GLabel 960  1510 2    47   Input ~ 0
+CE
+Text GLabel 960  1810 2    47   Input ~ 0
+MOSI
+Text GLabel 960  1910 2    47   Input ~ 0
+CLK
+Text GLabel 960  2010 2    47   Input ~ 0
+5V
+Text GLabel 960  1610 2    47   Input ~ 0
+RESET
+Text GLabel 960  1710 2    47   Input ~ 0
+LED
 $EndSCHEMATC

Commit message: Too many untracked changes: LCD boards update and switch to KiCAD version 5
Update the Nokia LCD breakout boards
Add more KiCAD simulation projects
Update most projects to KiCAD version 5
Parts:
- C1: symbol C_Small -> Nokia1616_LCD-rescue:C_Small
- CONN1: symbol Nokia1616_LCD -> Nokia1616_LCD-rescue:Nokia1616_LCD
- P1, P2: footprint Pin_Headers:Pin_Header_Straight_1x08 -> Pin_Headers:Pin_Header_Straight_1x08_Pitch2.54mm; symbol CONN_01X08 -> Nokia1616_LCD-rescue:CONN_01X08
- Q1: symbol BC547_BEC_123 -> Nokia1616_LCD-rescue:BC547_BEC_123
- R1: symbol R -> Nokia1616_LCD-rescue:R
Changed lines of the file:
@@
-EESchema Schematic File Version 2
-LIBS:power
-LIBS:device
-LIBS:transistors
-LIBS:conn
-LIBS:linear
-LIBS:regul
-LIBS:74xx
-LIBS:cmos4000
-LIBS:adc-dac
-LIBS:memory
-LIBS:xilinx
-LIBS:microcontrollers
-LIBS:dsp
-LIBS:microchip
-LIBS:analog_switches
-LIBS:motorola
-LIBS:texas
-LIBS:intel
-LIBS:audio
-LIBS:interface
-LIBS:digital-audio
-LIBS:philips
-LIBS:display
-LIBS:cypress
-LIBS:siliconi
-LIBS:opto
-LIBS:atmel
-LIBS:contrib
-LIBS:valves
+EESchema Schematic File Version 4
 LIBS:Nokia1616_LCD-cache
-EELAYER 25 0
+EELAYER 29 0
 EELAYER END
 $Descr User 5512 4331
@@
 Sheet 1 1
 Title "Nokia Color TFT LCD"
-Date "2017-01-29"
-Rev "1"
-Comp "Discovery Center"
-Comment1 "karibe.co"
+Date "2019-01-12"
+Rev "1.1"
+Comp "Karibe (K) Ltd"
+Comment1 "karibe.co.ke"
 Comment2 "@muriukidavid"
-Comment3 "Karibe David"
-Comment4 ""
+Comment3 ""
+Comment4 "Design by: Karibe David"
 $EndDescr
 $Comp
-L CONN_01X08 P1
+L Nokia1616_LCD-rescue:CONN_01X08 P1
 U 1 1 588CF000
 P 1410 1660
 F 0 "P1" H 1410 2110 50  0000 C CNN
 F 1 "CONN_01X08" V 1510 1660 50  0000 C CNN
-F 2 "Pin_Headers:Pin_Header_Straight_1x08" H 1410 1660 50  0001 C CNN
+F 2 "Pin_Headers:Pin_Header_Straight_1x08_Pitch2.54mm" H 1410 1660 50  0001 C CNN
 F 3 "" H 1410 1660 50  0000 C CNN
 	1    1410 1660
@@
 $EndComp
 $Comp
-L Nokia1616_LCD CONN1
+L Nokia1616_LCD-rescue:Nokia1616_LCD CONN1
 U 1 1 588CF2E5
 P 3080 1640
-F 0 "CONN1" H 3080 890 60  0000 C CNN
+F 0 "CONN1" H 2950 1030 60  0000 C CNN
 F 1 "Nokia1616_LCD" H 3090 2225 60  0000 C CNN
 F 2 "Connect:Nokia1616_LCD" H 3180 1640 60  0001 C CNN
@@
 GND
 $Comp
-L C_Small C1
+L Nokia1616_LCD-rescue:C_Small C1
 U 1 1 588CF578
 P 2390 1930
@@
 $EndComp
 Wire Wire Line
-	2560 2030 2390 2030
+	2560 2030 2460 2030
 Wire Wire Line
-	2390 2130 2560 2130
+	2390 2130 2460 2130
 Wire Wire Line
 	2460 2130 2460 2030
@@
 	2480 1850 2480 1830
 Wire Wire Line
-	2480 1830 2390 1830
+	2480 1830 2440 1830
 Wire Wire Line
-	2380 1750 2560 1750
+	2380 1750 2440 1750
 Wire Wire Line
 	2440 1750 2440 1830
@@
 LED
 $Comp
-L BC547_BEC_123 Q1
+L Nokia1616_LCD-rescue:BC547_BEC_123 Q1
 U 1 1 58C99E38
 P 4515 1925
@@
 LED
 $Comp
-L R R1
+L Nokia1616_LCD-rescue:R R1
 U 1 1 58C9A3B8
 P 4165 1925
@@
 $EndComp
 $Comp
-L CONN_01X08 P2
+L Nokia1616_LCD-rescue:CONN_01X08 P2
 U 1 1 58D4DEA8
 P 760 1660
 F 0 "P2" H 760 2110 50  0000 C CNN
 F 1 "CONN_01X08" V 860 1660 50  0000 C CNN
-F 2 "Pin_Headers:Pin_Header_Straight_1x08" H 760 1660 50  0001 C CNN
+F 2 "Pin_Headers:Pin_Header_Straight_1x08_Pitch2.54mm" H 760 1660 50  0001 C CNN
 F 3 "" H 760 1660 50  0000 C CNN
 	1    760  1660
@@
 Text GLabel 960  1710 2    47   Input ~ 0
 LED
+Wire Wire Line
+	2460 2030 2390 2030
+Wire Wire Line
+	2460 2130 2560 2130
+Wire Wire Line
+	2440 1830 2390 1830
+Wire Wire Line
+	2440 1750 2560 1750
 $EndSCHEMATC
