File: pogo/swd_pogo.sch (KiCad schematic (older format))
At the start: 4 parts, among them J1 CONN_02X05, J2 Conn_02x04_Odd_Even, J3 CONN_01X04, J4 CONN_01X04

Commit message: Too many untracked changes: LCD boards update and switch to KiCAD version 5
Update the Nokia LCD breakout boards
Add more KiCAD simulation projects
Update most projects to KiCAD version 5
Parts:
- added C1: 100nF, Capacitor_SMD:C_0402_1005Metric, symbol Device:C_Small
- added R1, R2: 10K, Resistor_SMD:R_0402_1005Metric, symbol Device:R_Small
- J1: symbol CONN_02X05 -> swd_pogo-rescue:CONN_02X05
- J2: symbol Conn_02x04_Odd_Even -> swd_pogo-rescue:Conn_02x04_Odd_Even
- J3, J4: symbol CONN_01X04 -> swd_pogo-rescue:CONN_01X04
Connections:
- net 3v3: now also R1.1, R2.2
- net GND: now also C1.2
- net RESET: now also C1.1, R2.1
- net SWDIO: now also R1.2
Other:
- moved on the sheet: J1, J2, J3, J4
Changed lines of the file:
@@
-EESchema Schematic File Version 2
-LIBS:power
-LIBS:device
-LIBS:transistors
-LIBS:conn
-LIBS:linear
-LIBS:regul
-LIBS:74xx
-LIBS:cmos4000
-LIBS:adc-dac
-LIBS:memory
-LIBS:xilinx
-LIBS:microcontrollers
-LIBS:dsp
-LIBS:microchip
-LIBS:analog_switches
-LIBS:motorola
-LIBS:texas
-LIBS:intel
-LIBS:audio
-LIBS:interface
-LIBS:digital-audio
-LIBS:philips
-LIBS:display
-LIBS:cypress
-LIBS:siliconi
-LIBS:opto
-LIBS:atmel
-LIBS:contrib
-LIBS:valves
-LIBS:swd_pogo-cache
-EELAYER 25 0
+EESchema Schematic File Version 4
+EELAYER 30 0
 EELAYER END
 $Descr User 5315 4000
 encoding utf-8
 Sheet 1 1
-Title "1.27mm 10 pin SWD to pogo adapter"
-Date "2017-09-07"
+Title "1.27mm 10 pin SWD to 8 pin pogo adapter"
+Date "2020-08-31"
 Rev "1"
-Comp "Sign-IO"
+Comp "Karibe (K) Ltd"
 Comment1 "@muriukidavid"
 Comment2 ""
@@
 $EndDescr
 $Comp
-L CONN_02X05 J1
+L swd_pogo-rescue:CONN_02X05 J1
 U 1 1 59B05100
-P 1300 1500
-F 0 "J1" H 1300 1800 50  0000 C CNN
-F 1 "CONN_02X05" H 1300 1200 50  0000 C CNN
-F 2 "Pin_Headers:Pin_Header_Straight_2x05_Pitch1.27mm" H 1300 300 50  0001 C CNN
-F 3 "" H 1300 300 50  0001 C CNN
-	1    1300 1500
+P 1200 1400
+F 0 "J1" H 1200 1700 50  0000 C CNN
+F 1 "CONN_02X05" H 1200 1100 50  0000 C CNN
+F 2 "Pin_Headers:Pin_Header_Straight_2x05_Pitch1.27mm" H 1200 200 50  0001 C CNN
+F 3 "" H 1200 200 50  0001 C CNN
+	1    1200 1400
 	1    0    0    -1
 $EndComp
-Text GLabel 1550 1700 2    24   Input ~ 0
+Text GLabel 1550 1600 2    39   Input ~ 0
 RESET
-Text GLabel 1550 1400 2    24   Input ~ 0
+Text GLabel 1450 1300 2    39   Input ~ 0
 SWDCLK
-Text GLabel 1550 1300 2    24   Input ~ 0
+Text GLabel 1450 1200 2    39   Input ~ 0
 SWDIO
-Text GLabel 1550 1500 2    24   Input ~ 0
+Text GLabel 1450 1400 2    39   Input ~ 0
 SWDTRACE
-Text GLabel 2925 1350 0    24   Input ~ 0
+Text GLabel 3125 1350 0    39   Input ~ 0
 3v3
-Text GLabel 1050 1300 0    24   Input ~ 0
+Text GLabel 950  1200 0    39   Input ~ 0
 3v3
-Text GLabel 1050 1500 0    24   Input ~ 0
+Text GLabel 950  1400 0    39   Input ~ 0
 GND
-Text GLabel 1050 1400 0    24   Input ~ 0
+Text GLabel 950  1300 0    39   Input ~ 0
 GND
-Text GLabel 1050 1600 0    24   Input ~ 0
+Text GLabel 950  1500 0    39   Input ~ 0
 UARTTX
-Text GLabel 1550 1600 2    24   Input ~ 0
+Text GLabel 1450 1500 2    39   Input ~ 0
 UARTRX
-Text GLabel 1050 1700 0    24   Input ~ 0
+Text GLabel 950  1600 0    39   Input ~ 0
 GNDDETECT
-Text GLabel 3425 1550 2    24   Input ~ 0
+Text GLabel 3625 1550 2    39   Input ~ 0
 GND
-Text GLabel 2925 1450 0    24   Input ~ 0
+Text GLabel 3125 1450 0    39   Input ~ 0
 SWDCLK
-Text GLabel 2925 1550 0    24   Input ~ 0
+Text GLabel 3125 1550 0    39   Input ~ 0
 RESET
-Text GLabel 3425 1450 2    24   Input ~ 0
+Text GLabel 3625 1450 2    39   Input ~ 0
 SWDTRACE
 $Comp
-L CONN_01X04 J3
+L swd_pogo-rescue:CONN_01X04 J3
 U 1 1 59B0E8DD
-P 2150 1500
-F 0 "J3" H 2150 1750 50  0000 C CNN
-F 1 "CONN_01X04" V 2250 1500 50  0000 C CNN
-F 2 "Pin_Headers:Pin_Header_Straight_01x04_Pitch1.27mm_wide" H 2150 1500 50  0001 C CNN
-F 3 "" H 2150 1500 50  0001 C CNN
-	1    2150 1500
+P 2100 1500
+F 0 "J3" H 2100 1750 50  0000 C CNN
+F 1 "CONN_01X04" V 2200 1500 50  0000 C CNN
+F 2 "Pin_Headers:Pin_Header_Straight_01x04_Pitch1.27mm_wide" H 2100 1500 50  0001 C CNN
+F 3 "" H 2100 1500 50  0001 C CNN
+	1    2100 1500
 	-1   0    0    -1
 $EndComp
 $Comp
-L CONN_01X04 J4
+L swd_pogo-rescue:CONN_01X04 J4
 U 1 1 59B0EBBC
-P 4150 1500
-F 0 "J4" H 4150 1750 50  0000 C CNN
-F 1 "CONN_01X04" V 4250 1500 50  0000 C CNN
-F 2 "Pin_Headers:Pin_Header_Straight_01x04_Pitch1.27mm_wide" H 4150 1500 50  0001 C CNN
-F 3 "" H 4150 1500 50  0001 C CNN
-	1    4150 1500
+P 4500 1500
+F 0 "J4" H 4500 1750 50  0000 C CNN
+F 1 "CONN_01X04" V 4600 1500 50  0000 C CNN
+F 2 "Pin_Headers:Pin_Header_Straight_01x04_Pitch1.27mm_wide" H 4500 1500 50  0001 C CNN
+F 3 "" H 4500 1500 50  0001 C CNN
+	1    4500 1500
 	1    0    0    -1
 $EndComp
-Text GLabel 2350 1350 2    24   Input ~ 0
+Text GLabel 2400 1350 2    39   Input ~ 0
 SWDIO
-Text GLabel 2350 1450 2    24   Input ~ 0
+Text GLabel 2300 1450 2    39   Input ~ 0
 SWDCLK
-Text GLabel 2350 1550 2    24   Input ~ 0
+Text GLabel 2300 1550 2    39   Input ~ 0
 SWDTRACE
-Text GLabel 3950 1350 0    24   Input ~ 0
+Text GLabel 4300 1350 0    39   Input ~ 0
 3v3
-Text GLabel 2350 1650 2    24   Input ~ 0
+Text GLabel 2400 1650 2    39   Input ~ 0
 RESET
-Text GLabel 3950 1650 0    24   Input ~ 0
+Text GLabel 4300 1650 0    39   Input ~ 0
 UARTTX
-Text GLabel 3950 1450 0    24   Input ~ 0
+Text GLabel 4300 1450 0    39   Input ~ 0
 GND
-Text GLabel 3950 1550 0    24   Input ~ 0
+Text GLabel 4300 1550 0    39   Input ~ 0
 UARTRX
-Text GLabel 3425 1350 2    24   Input ~ 0
+Text GLabel 3625 1350 2    39   Input ~ 0
 SWDIO
 $Comp
-L Conn_02x04_Odd_Even J2
+L swd_pogo-rescue:Conn_02x04_Odd_Even J2
 U 1 1 59D3A2DD
-P 3125 1450
-F 0 "J2" H 3175 1650 50  0000 C CNN
-F 1 "Conn_02x04_Odd_Even" H 3175 1150 50  0000 C CNN
-F 2 "Pin_Headers:Pin_Header_Pogo_02x04_Pitch1.27mm" H 3125 1450 50  0001 C CNN
-F 3 "" H 3125 1450 50  0001 C CNN
-	1    3125 1450
+P 3325 1450
+F 0 "J2" H 3375 1650 50  0000 C CNN
+F 1 "Conn_02x04_Odd_Even" H 3375 1150 50  0000 C CNN
+F 2 "Pin_Headers:Pin_Header_Pogo_02x04_Pitch1.27mm" H 3325 1450 50  0001 C CNN
+F 3 "" H 3325 1450 50  0001 C CNN
+	1    3325 1450
 	1    0    0    -1
 $EndComp
-Text GLabel 2925 1650 0    24   Input ~ 0
+Text GLabel 3125 1650 0    39   Input ~ 0
 UARTRX
-Text GLabel 3425 1650 2    24   Input ~ 0
+Text GLabel 3625 1650 2    39   Input ~ 0
 UARTTX
+$Comp
+L Device:C_Small C1
+U 1 1 5F4CFFAF
+P 1500 1750
+F 0 "C1" H 1592 1796 50  0000 L CNN
+F 1 "100nF" H 1592 1705 50  0000 L CNN
+F 2 "Capacitor_SMD:C_0402_1005Metric" H 1500 1750 50  0001 C CNN
+F 3 "~" H 1500 1750 50  0001 C CNN
+	1    1500 1750
+	1    0    0    -1
+$EndComp
+$Comp
+L power:GND #PWR0101
+U 1 1 5F4D0361
+P 1500 1850
+F 0 "#PWR0101" H 1500 1600 50  0001 C CNN
+F 1 "GND" H 1505 1677 50  0000 C CNN
+F 2 "" H 1500 1850 50  0001 C CNN
+F 3 "" H 1500 1850 50  0001 C CNN
+	1    1500 1850
+	1    0    0    -1
+$EndComp
+Wire Wire Line
+	1450 1600 1500 1600
+Wire Wire Line
+	1500 1650 1500 1600
+Connection ~ 1500 1600
+Wire Wire Line
+	1500 1600 1550 1600
+$Comp
+L Device:R_Small R2
+U 1 1 5F4D0919
+P 2350 1800
+F 0 "R2" H 2409 1846 50  0000 L CNN
+F 1 "10K" H 2409 1755 50  0000 L CNN
+F 2 "Resistor_SMD:R_0402_1005Metric" H 2350 1800 50  0001 C CNN
+F 3 "~" H 2350 1800 50  0001 C CNN
+	1    2350 1800
+	1    0    0    -1
+$EndComp
+Wire Wire Line
+	2300 1650 2350 1650
+Wire Wire Line
+	2350 1700 2350 1650
+Connection ~ 2350 1650
+Wire Wire Line
+	2350 1650 2400 1650
+Text GLabel 2300 1950 0    39   Input ~ 0
+3v3
+Wire Wire Line
+	2300 1950 2350 1950
+Wire Wire Line
+	2350 1950 2350 1900
+$Comp
+L Device:R_Small R1
+U 1 1 5F4D14DA
+P 2350 1200
+F 0 "R1" H 2409 1246 50  0000 L CNN
+F 1 "10K" H 2409 1155 50  0000 L CNN
+F 2 "Resistor_SMD:R_0402_1005Metric" H 2350 1200 50  0001 C CNN
+F 3 "~" H 2350 1200 50  0001 C CNN
+	1    2350 1200
+	1    0    0    -1
+$EndComp
+Wire Wire Line
+	2300 1350 2350 1350
+Wire Wire Line
+	2350 1300 2350 1350
+Connection ~ 2350 1350
+Wire Wire Line
+	2350 1350 2400 1350
+Text GLabel 2350 1100 1    39   Input ~ 0
+3v3
 $EndSCHEMATC
